Commit message: Fix: minor fix

File: config/Z-Arm_10042C0.ros2_control.xacro (robot description, xacro)
@@ -2,5 +2,5 @@
 <robot xmlns:xacro="http://www.ros.org/wiki/xacro">
     <xacro:macro name="Z-Arm_10042C0_ros2_control" params="name initial_positions_file">
-        <xacro:property name="initial_positions" value="${load_yaml(initial_positions_file)['initial_positions']}"/>
+        <xacro:property name="initial_positions" value="${xacro.load_yaml(initial_positions_file)['initial_positions']}"/>
         <ros2_control name="${name}" type="system">
             <hardware>
@@ -8,8 +8,4 @@
                 <plugin>mock_components/GenericSystem</plugin>
             </hardware>
-        <!-- <ros2_control name="GazeboSystem" type="system">
-			<hardware>
-				<plugin>gazebo_ros2_control/GazeboSystem</plugin>
-	    	</hardware> -->
             <joint name="joint1">
                 <command_interface name="position"/>
